Commit message: update code

File: install/rmitbot_description/share/rmitbot_description/urdf/rmitbot.urdf.xacro (robot description, xacro)
@@ -1,9 +1 @@
-<?xml version="1.0"?>
-<!-- This is the main urdf document, calling other xacro, including -->
-<!-- rmitbot_platform:  main platform -->
-<!-- rmitbot_gazebo:    gazebo simulation parameters for the main platform -->
-<robot name="rmitbot"
-    xmlns:xacro="http://ros.org/wiki/xacro">
-    <xacro:include filename="$(find rmitbot_description)/urdf/rmitbot_platform.xacro" />
-    <xacro:include filename="$(find rmitbot_description)/urdf/rmitbot_gazebo.xacro" />
-</robot>
+/home/v120506/03-ROS2_Workspace/rmitbot_v5/lesson1_ws/src/rmitbot_description/urdf/rmitbot.urdf.xacro

File: install/rmitbot_description/share/rmitbot_description/urdf/rmitbot_gazebo.xacro (robot description, xacro)
@@ -1,63 +1 @@
-<?xml version="1.0"?>
-<!-- Gazebo file contains information regarding the lnks's physics (e.g., friction, stiffness, damping) -->
-<robot name="rmitbot" xmlns:xacro="http://ros.org/wiki/xacro" xmlns:gz="http://gazebosim.org/schema">
-  <!-- Wheels -->
-     <!-- To emulate Mecanum wheels in Gazebo with spherical collisions it
-  requires a custom friction model so the vehicle can strafe left to right -->
-  <gazebo reference='front_left_wheel'>
-    <collision>
-      <surface>
-        <friction>
-          <ode>
-            <mu>1.0</mu>
-            <mu2>0.0</mu2>
-            <!-- <fdir1 gz:expressed_in="base_link">1 -1 0</fdir1> -->
-            <fdir1 gz:expressed_in="base_footprint">1 -1 0</fdir1>
-          </ode>
-        </friction>
-      </surface>
-    </collision>
-  </gazebo>
-  <gazebo reference='front_right_wheel'>
-    <collision>
-      <surface>
-        <friction>
-          <ode>
-            <mu>1.0</mu>
-            <mu2>0.0</mu2>
-            <!-- <fdir1 gz:expressed_in="base_link">1 1 0</fdir1> -->
-            <fdir1 gz:expressed_in="base_footprint">1 1 0</fdir1>
-          </ode>
-        </friction>
-      </surface>
-    </collision>
-  </gazebo>
-  <gazebo reference='rear_left_wheel'>
-    <collision>
-      <surface>
-        <friction>
-          <ode>
-            <mu>1.0</mu>
-            <mu2>0.0</mu2>
-            <!-- <fdir1 gz:expressed_in="base_link">1 1 0</fdir1> -->
-            <fdir1 gz:expressed_in="base_footprint">1 1 0</fdir1>
-          </ode>
-        </friction>
-      </surface>
-    </collision>
-  </gazebo>
-  <gazebo reference='rear_right_wheel'>
-    <collision>
-      <surface>
-        <friction>
-          <ode>
-            <mu>1.0</mu>
-            <mu2>0.0</mu2>
-            <!-- <fdir1 gz:expressed_in="base_link">1 -1 0</fdir1> -->
-            <fdir1 gz:expressed_in="base_footprint">1 -1 0</fdir1>
-          </ode>
-        </friction>
-      </surface>
-    </collision>
-  </gazebo>
-</robot>
+/home/v120506/03-ROS2_Workspace/rmitbot_v5/lesson1_ws/src/rmitbot_description/urdf/rmitbot_gazebo.xacro

File: install/rmitbot_description/share/rmitbot_description/urdf/rmitbot_platform.xacro (robot description, xacro)
@@ -1,189 +1 @@
-<?xml version="1.0"?>
-<robot name="rmitbot" xmlns:xacro="http://www.ros.org/wiki/xacro" xmlns:gz="http://gazebosim.org/schema">
-  <material name="orange">
-    <color rgba="0.8 0.4 0.0 1.0" />
-  </material>
-  <material name="black">
-    <color rgba="0.5 0.5 0.5 1.0" />
-  </material>
-  <material name="white">
-    <color rgba="1 1 1 1.0" />
-  </material>
-  <link name="base_footprint" />
-  <joint name="base_joint" type="fixed">
-    <parent link="base_footprint" />
-    <child link="base_link" />
-    <origin xyz="0 0 0.05" rpy="0 0 0" />
-  </joint>
-  <!-- Base Link -->
-  <link name="base_link">
-    <collision>
-      <origin xyz="0 0 0.05" rpy="0 0 0" />
-      <geometry>
-         <box size=".28 .3 0.1" />
-      </geometry>
-    </collision>
-    <visual>
-      <origin xyz="0 0 0.05" rpy="0 0 0" />
-      <geometry>
-         <box size=".28 .3 0.1" />
-      </geometry>
-      <material name="orange" />
-    </visual>
-    <inertial>
-      <origin xyz="0 0 0.5" rpy="0 0 0" />
-      <mass value="1.5" />
-      <inertia
-        ixx="0.13"
-        ixy="0.0"
-        ixz="0.0"
-        iyy="0.42"
-        iyz="0.0"
-        izz="0.48" />
-    </inertial>
-  </link>
-  <!-- front left wheel -->
-  <joint name="front_left_wheel_joint" type="continuous">
-    <origin xyz="0.14 0.15 0" rpy="-${pi/2} 0 0" />
-    <parent link="base_link" />
-    <child link="front_left_wheel" />
-    <axis xyz="0 0 1" />
-    <dynamics damping="0.2" />
-  </joint>
-  <link name="front_left_wheel">
-    <collision>
-      <!-- <origin xyz="0 0 .06" rpy="0 0 0" /> -->
-      <origin xyz="0 0 .025" rpy="0 0 0" />
-      <geometry>
-        <sphere radius="0.05" />
-      </geometry>
-    </collision>
-    <visual>
-      <!-- <origin xyz="0 0 .06" rpy="0 0 0" /> -->
-      <origin xyz="0 0 .025" rpy="0 0 0" />
-      <geometry>
-        <!-- <sphere radius="0.3" /> -->
-        <cylinder radius="0.05" length="0.05" />
-      </geometry>
-      <material name="black" />
-    </visual>
-    <inertial>
-      <!-- <origin xyz="0 0 .06" rpy="0 0 0" /> -->
-       <origin xyz="0 0 .025" rpy="0 0 0" />
-      <mass value="0.5" />
-      <inertia ixx="0.0025"
-        ixy="0.0"
-        ixz="0.0"
-        iyy="0.0025"
-        iyz="0.0"
-        izz="0.0020" />
-    </inertial>
-  </link>
-  <!-- front right wheel -->
-  <joint name="front_right_wheel_joint" type="continuous">
-    <origin xyz="0.14 -0.15 0." rpy="-${pi/2} 0 0" />
-    <parent link="base_link" />
-    <child link="front_right_wheel" />
-    <axis xyz="0 0 1" />
-    <dynamics damping="0.2" />
-  </joint>
-  <link name="front_right_wheel">
-    <collision>
-      <!-- <origin xyz="0 0 -.06" rpy="0 0 0" /> -->
-      <origin xyz="0 0 -.025" rpy="0 0 0" />
-      <geometry>
-        <sphere radius="0.05" />
-      </geometry>
-    </collision>
-    <visual>
-      <origin xyz="0 0 -.025" rpy="0 0 0" />
-      <geometry>
-        <cylinder radius="0.05" length="0.05" />
-      </geometry>
-      <material name="black" />
-    </visual>
-    <inertial>
-      <!-- <origin xyz="0 0 -.06" rpy="0 0 0" /> -->
-      <origin xyz="0 0 -.025" rpy="0 0 0" />
-      <mass value=".5" />
-      <inertia ixx="0.0025"
-        ixy="0.0"
-        ixz="0.0"
-        iyy="0.0025"
-        iyz="0.0"
-        izz="0.0020" />
-    </inertial>
-  </link>
-  <!-- rear left wheel -->
-  <joint name="rear_left_wheel_joint" type="continuous">
-    <origin xyz="-0.14 0.15 0." rpy="-${pi/2} 0 0" />
-    <parent link="base_link" />
-    <child link="rear_left_wheel" />
-    <axis xyz="0 0 1" />
-    <dynamics damping="0.2" />
-  </joint>
-  <link name="rear_left_wheel">
-    <collision>
-      <!-- <origin xyz="0 0 .06" rpy="0 0 0" /> -->
-       <origin xyz="0 0 .025" rpy="0 0 0" />
-      <geometry>
-        <sphere radius="0.05" />
-      </geometry>
-    </collision>
-    <visual>
-      <!-- <origin xyz="0 0 .06" rpy="0 0 0" /> -->
-       <origin xyz="0 0 .025" rpy="0 0 0" />
-      <geometry>
-        <cylinder radius="0.05" length="0.05" />
-      </geometry>
-      <material name="black" />
-    </visual>
-    <inertial>
-      <!-- <origin xyz="0 0 .06" rpy="0 0 0" /> -->
-       <origin xyz="0 0 .025" rpy="0 0 0" />
-      <mass value="0.5" />
-      <inertia ixx="0.0025"
-        ixy="0.0"
-        ixz="0.0"
-        iyy="0.0025"
-        iyz="0.0"
-        izz="0.0020" />
-    </inertial>
-  </link>
-  <!-- rear right wheel -->
-  <joint name="rear_right_wheel_joint" type="continuous">
-    <origin xyz="-0.14 -0.15 0." rpy="-${pi/2} 0 0" />
-    <parent link="base_link" />
-    <child link="rear_right_wheel" />
-    <axis xyz="0 0 1" />
-    <dynamics damping="0.2" />
-  </joint>
-  <link name="rear_right_wheel">
-    <collision>
-      <!-- <origin xyz="0 0 -.06" rpy="0 0 0" /> -->
-       <origin xyz="0 0 -.025" rpy="0 0 0" />
-      <geometry>
-        <sphere radius="0.05" />
-      </geometry>
-    </collision>
-    <visual>
-      <!-- <origin xyz="0 0 -.06" rpy="0 0 0" /> -->
-       <origin xyz="0 0 -.025" rpy="0 0 0" />
-      <geometry>
-        <cylinder radius="0.05" length="0.05" />
-      </geometry>
-      <material name="black" />
-    </visual>
-    <inertial>
-      <!-- <origin xyz="0 0 -.06" rpy="0 0 0" /> -->
-       <origin xyz="0 0 -.025" rpy="0 0 0" />
-      <mass value="0.5" />
-      <inertia ixx="0.0025"
-        ixy="0.0"
-        ixz="0.0"
-        iyy="0.0025"
-        iyz="0.0"
-        izz="0.0020" />
-    </inertial>
-  </link>
-</robot>
+/home/v120506/03-ROS2_Workspace/rmitbot_v5/lesson1_ws/src/rmitbot_description/urdf/rmitbot_platform.xacro

File: src/rmitbot_description/urdf/rmitbot.urdf.xacro (robot description, xacro)
@@ -3,7 +3,7 @@
 <!-- rmitbot_platform:  main platform -->
 <!-- rmitbot_gazebo:    gazebo simulation parameters for the main platform -->
-<robot name="rmitbot"
-    xmlns:xacro="http://ros.org/wiki/xacro">
+<robot name="rmitbot" xmlns:xacro="http://ros.org/wiki/xacro">
+    <xacro:include filename="$(find rmitbot_description)/urdf/common_properties.xacro" />
     <xacro:include filename="$(find rmitbot_description)/urdf/rmitbot_platform.xacro" />
-    <xacro:include filename="$(find rmitbot_description)/urdf/rmitbot_gazebo.xacro" />
+    <xacro:include filename="$(find rmitbot_description)/urdf/rmitbot_wheel.xacro" />
 </robot>

File: src/rmitbot_description/urdf/rmitbot_platform.xacro (robot description, xacro)
@@ -1,20 +1,6 @@
 <?xml version="1.0"?>
 <robot name="rmitbot" xmlns:xacro="http://www.ros.org/wiki/xacro" xmlns:gz="http://gazebosim.org/schema">
-  <material name="orange">
-    <color rgba="0.8 0.4 0.0 1.0" />
-  </material>
-  <material name="black">
-    <color rgba="0.5 0.5 0.5 1.0" />
-  </material>
-  <material name="white">
-    <color rgba="1 1 1 1.0" />
-  </material>
   <link name="base_footprint" />
-  <joint name="base_joint" type="fixed">
-    <parent link="base_footprint" />
-    <child link="base_link" />
-    <origin xyz="0 0 0.05" rpy="0 0 0" />
-  </joint>
-  <!-- Base Link -->
+  <!-- Inertial, visual, collision of the link -->
   <link name="base_link">
     <collision>
@@ -43,147 +29,9 @@
     </inertial>
   </link>
-  <!-- front left wheel -->
-  <joint name="front_left_wheel_joint" type="continuous">
-    <origin xyz="0.14 0.15 0" rpy="-${pi/2} 0 0" />
-    <parent link="base_link" />
-    <child link="front_left_wheel" />
-    <axis xyz="0 0 1" />
-    <dynamics damping="0.2" />
+  <!-- Parent, child, and origin -->
+  <joint name="base_joint" type="fixed">
+    <parent link="base_footprint" />
+    <child link="base_link" />
+    <origin xyz="0 0 0.05" rpy="0 0 0" />
   </joint>
-  <link name="front_left_wheel">
-    <collision>
-      <!-- <origin xyz="0 0 .06" rpy="0 0 0" /> -->
-      <origin xyz="0 0 .025" rpy="0 0 0" />
-      <geometry>
-        <sphere radius="0.05" />
-      </geometry>
-    </collision>
-    <visual>
-      <!-- <origin xyz="0 0 .06" rpy="0 0 0" /> -->
-      <origin xyz="0 0 .025" rpy="0 0 0" />
-      <geometry>
-        <!-- <sphere radius="0.3" /> -->
-        <cylinder radius="0.05" length="0.05" />
-      </geometry>
-      <material name="black" />
-    </visual>
-    <inertial>
-      <!-- <origin xyz="0 0 .06" rpy="0 0 0" /> -->
-       <origin xyz="0 0 .025" rpy="0 0 0" />
-      <mass value="0.5" />
-      <inertia ixx="0.0025"
-        ixy="0.0"
-        ixz="0.0"
-        iyy="0.0025"
-        iyz="0.0"
-        izz="0.0020" />
-    </inertial>
-  </link>
-  <!-- front right wheel -->
-  <joint name="front_right_wheel_joint" type="continuous">
-    <origin xyz="0.14 -0.15 0." rpy="-${pi/2} 0 0" />
-    <parent link="base_link" />
-    <child link="front_right_wheel" />
-    <axis xyz="0 0 1" />
-    <dynamics damping="0.2" />
-  </joint>
-  <link name="front_right_wheel">
-    <collision>
-      <!-- <origin xyz="0 0 -.06" rpy="0 0 0" /> -->
-      <origin xyz="0 0 -.025" rpy="0 0 0" />
-      <geometry>
-        <sphere radius="0.05" />
-      </geometry>
-    </collision>
-    <visual>
-      <origin xyz="0 0 -.025" rpy="0 0 0" />
-      <geometry>
-        <cylinder radius="0.05" length="0.05" />
-      </geometry>
-      <material name="black" />
-    </visual>
-    <inertial>
-      <!-- <origin xyz="0 0 -.06" rpy="0 0 0" /> -->
-      <origin xyz="0 0 -.025" rpy="0 0 0" />
-      <mass value=".5" />
-      <inertia ixx="0.0025"
-        ixy="0.0"
-        ixz="0.0"
-        iyy="0.0025"
-        iyz="0.0"
-        izz="0.0020" />
-    </inertial>
-  </link>
-  <!-- rear left wheel -->
-  <joint name="rear_left_wheel_joint" type="continuous">
-    <origin xyz="-0.14 0.15 0." rpy="-${pi/2} 0 0" />
-    <parent link="base_link" />
-    <child link="rear_left_wheel" />
-    <axis xyz="0 0 1" />
-    <dynamics damping="0.2" />
-  </joint>
-  <link name="rear_left_wheel">
-    <collision>
-      <!-- <origin xyz="0 0 .06" rpy="0 0 0" /> -->
-       <origin xyz="0 0 .025" rpy="0 0 0" />
-      <geometry>
-        <sphere radius="0.05" />
-      </geometry>
-    </collision>
-    <visual>
-      <!-- <origin xyz="0 0 .06" rpy="0 0 0" /> -->
-       <origin xyz="0 0 .025" rpy="0 0 0" />
-      <geometry>
-        <cylinder radius="0.05" length="0.05" />
-      </geometry>
-      <material name="black" />
-    </visual>
-    <inertial>
-      <!-- <origin xyz="0 0 .06" rpy="0 0 0" /> -->
-       <origin xyz="0 0 .025" rpy="0 0 0" />
-      <mass value="0.5" />
-      <inertia ixx="0.0025"
-        ixy="0.0"
-        ixz="0.0"
-        iyy="0.0025"
-        iyz="0.0"
-        izz="0.0020" />
-    </inertial>
-  </link>
-  <!-- rear right wheel -->
-  <joint name="rear_right_wheel_joint" type="continuous">
-    <origin xyz="-0.14 -0.15 0." rpy="-${pi/2} 0 0" />
-    <parent link="base_link" />
-    <child link="rear_right_wheel" />
-    <axis xyz="0 0 1" />
-    <dynamics damping="0.2" />
-  </joint>
-  <link name="rear_right_wheel">
-    <collision>
-      <!-- <origin xyz="0 0 -.06" rpy="0 0 0" /> -->
-       <origin xyz="0 0 -.025" rpy="0 0 0" />
-      <geometry>
-        <sphere radius="0.05" />
-      </geometry>
-    </collision>
-    <visual>
-      <!-- <origin xyz="0 0 -.06" rpy="0 0 0" /> -->
-       <origin xyz="0 0 -.025" rpy="0 0 0" />
-      <geometry>
-        <cylinder radius="0.05" length="0.05" />
-      </geometry>
-      <material name="black" />
-    </visual>
-    <inertial>
-      <!-- <origin xyz="0 0 -.06" rpy="0 0 0" /> -->
-       <origin xyz="0 0 -.025" rpy="0 0 0" />
-      <mass value="0.5" />
-      <inertia ixx="0.0025"
-        ixy="0.0"
-        ixz="0.0"
-        iyy="0.0025"
-        iyz="0.0"
-        izz="0.0020" />
-    </inertial>
-  </link>
 </robot>
